File: Design/wearable_device/wearable_device.kicad_sch (KiCad schematic)
At the start: 3 parts, among them IC1 TESEO-LIV3R, U1 ESP32-S3-MINI-1, U2 MAX30102

Commit message: complete design pcb board
Parts:
- removed IC1: TESEO-LIV3R, TESEOLIV3R, symbol SamacSys_Parts:TESEO-LIV3R
- removed U2: MAX30102, OptoDevice:Maxim_OLGA-14_3.3x5.6mm_P0.8mm, symbol Sensor:MAX30102
- added C1, C13, C14, C17, C2, C3, C6, C8: 10uF, Capacitor_SMD:C_0603_1608Metric, symbol Device:C
- added C12: 10nF, Capacitor_SMD:C_0603_1608Metric, symbol Device:C
- added C15, C16: 100nF, Capacitor_SMD:C_0603_1608Metric, symbol Device:C
- added C4, C5, C7, C9: 0.1uF, Capacitor_SMD:C_0603_1608Metric, symbol Device:C
- added J1: Micro_SD_Card, Connector_Card:microSD_HC_Hirose_DM3D-SF, symbol Connector:Micro_SD_Card
- added J2: POWER, Connector_PinHeader_2.00mm:PinHeader_1x01_P2.00mm_Vertical, symbol Connector:Conn_01x01_Pin
- added J3, J4: Conn_01x04_Pin, Connector_PinHeader_2.00mm:PinHeader_1x04_P2.00mm_Vertical, symbol Connector:Conn_01x04_Pin
- added J5: Conn_01x07_Pin, Connector_PinHeader_2.54mm:PinHeader_1x07_P2.54mm_Vertical, symbol Connector:Conn_01x07_Pin
- added J6: GND, Connector_PinHeader_2.00mm:PinHeader_1x01_P2.00mm_Vertical, symbol Connector:Conn_01x01_Pin
- added P1: USB_C_Plug_USB2.0, Connector_USB:USB_C_Receptacle_GCT_USB4105-xx-A_16P_TopMnt_Horizontal, symbol Connector:USB_C_Plug_USB2.0
- added Q1, Q2: BSS138, Package_TO_SOT_SMD:SOT-23, symbol Transistor_FET:BSS138
- added Q3, Q5: BC817, Package_TO_SOT_SMD:SOT-23, symbol Transistor_BJT:BC817
- added R1, R10, R11, R12, R13, R14, R15, R16, R2, R4, R5, R6, R7: 10k, Resistor_SMD:R_0603_1608Metric, symbol Device:R
- added R3: 1.2k, Resistor_SMD:R_0603_1608Metric, symbol Device:R
- added R8, R9: 4.7k, Resistor_SMD:R_0603_1608Metric, symbol Device:R
- added SW1: SW_Push, Button_Switch_SMD:SW_Tactile_SPST_NO_Straight_CK_PTS636Sx25SMTRLFS, symbol Switch:SW_Push
- added U2: L80-R, L80-R:XCVR_L80-R, symbol L80-R:L80-R
- added U3: LP2985-33DBVR, LP2985-33DBVR:SOT95P280X145-5N, symbol LP2985-33DBVR:LP2985-33DBVR
- added U4: TP4056, TP4056:SOP127P600X175-9N, symbol TP4056:TP4056
- added U5: LIS2DH12TR, LIS2DH12TR:PQFN50P200X200100-12N, symbol LIS2DH12TR:LIS2DH12TR
- added U6: CH340C, Package_SO:SOIC-16_3.9x9.9mm_P1.27mm, symbol Interface_USB:CH340C
Connections:
- net GND: now reaches U1.1 (GND), U1.2 (GND), U1.42 (GND), U1.43 (GND), U1.46 (GND), U1.47 (GND), U1.48 (GND), U1.49 (GND), U1.50 (GND), U1.51 (GND), U1.52 (GND), U1.53 (GND), U1.54 (GND), U1.55 (GND), U1.56 (GND), U1.57 (GND), U1.58 (GND), U1.59 (GND), U1.60 (GND), U1.61 (GND), U1.62 (GND), U1.63 (GND), U1.64 (GND), U1.65 (GND)
- net GND: now also C12.2, C13.2, C14.2, C15.2, C16.2, C17.2, C2.2, C3.2, C4.2, C5.2, C7.2, C8.2, C9.2, J1.6 (VSS), J1.9 (SHIELD), J3.1 (Pin_1), J4.4 (Pin_4), J5.1 (Pin_1), J6.1 (Pin_1), P1.A1 (GND), P1.A12 (GND), P1.B1 (GND), P1.B12 (GND), P1.S1 (SHIELD), Q1.2 (S), Q2.2 (S), R16.2, R3.2, U2.12 (GND), U2.3 (GND), U3.2 (GND), U4.1 (TEMP), U4.3 (GND), U5.5 (RES), U5.6 (GND), U5.7 (GND), U5.8 (GND), U6.1 (GND)
- net MOSI_SPI2: now reaches U1.10 (IO6)
- net MOSI_SPI2: now also J1.3 (CMD), R11.2
- net CS_SPI2: now reaches U1.11 (IO7)
- net CS_SPI2: now also J1.2 (DAT3/CD), R1.2
- net RES_TFT: now reaches U1.12 (IO8)
- net RES_TFT: now also J5.5 (Pin_5)
- net DC_TFT: now reaches U1.13 (IO9)
- net DC_TFT: now also J5.6 (Pin_6)
- net BLK_TFT: now reaches U1.14 (IO10)
- net BLK_TFT: now also J5.7 (Pin_7)
- net MOSI_TFT: now reaches U1.16 (IO12)
- net MOSI_TFT: now also J5.4 (Pin_4)
- net I2C_SCL: now reaches U1.17 (IO13)
- net I2C_SCL: now also J4.3 (Pin_3), R8.2, U5.1 (SCL/SPC)
- net I2C_SDA: now reaches U1.18 (IO14)
- net I2C_SDA: now also J4.2 (Pin_2), R9.2, U5.4 (SDA/SDI/SDO)
- net SCLK_TFT: now reaches U1.19 (IO15)
- net SCLK_TFT: now also J5.3 (Pin_3)
- net CLK_SPI2: now reaches U1.20 (IO16)
- net CLK_SPI2: now also J1.5 (CLK), R10.2
- net RXD1: now reaches U1.21 (IO17)
- net RXD1: now also U2.1 (RXD1)
- net TXD1: now reaches U1.22 (IO18)
- net TXD1: now also U2.2 (TXD1)
- net MISO_SPI2: now reaches U1.23 (IO19)
- net MISO_SPI2: now also J1.7 (DAT0), R12.2
- net +3.3V: now reaches U1.3 (3V3)
- net +3.3V: now also C1.2, C15.1, C16.1, C17.1, C3.1, C4.1, C5.1, C6.2, C7.1, C8.1, C9.1, J1.4 (VDD), J4.1 (Pin_1), J5.2 (Pin_2), R1.1, R10.1, R11.1, R12.1, R15.1, R2.1, R6.1, R7.1, R8.1, R9.1, SW1.1, U2.4 (VCC), U2.5 (V_BCKP), U3.5 (VOUT), U5.10 (VDD_IO), U5.2 (CS), U5.3 (SDO/SAO), U5.9 (VDD), U6.16 (VCC), U6.4 (V3)
- net SG_STDBY: now reaches U1.33 (IO37)
- net SG_STDBY: now also Q2.3 (D), R6.2
- net SG_CHRG: now reaches U1.34 (IO38)
- net SG_CHRG: now also Q1.3 (D), R7.2
- net BTN_CONTROL: now reaches U1.35 (IO39)
- net BTN_CONTROL: now also R16.1, SW1.2
- net at U1.39 (TXD0): now also U6.3 (RXD)
- net ESP32_IO0: now reaches U1.4 (IO0)
- net ESP32_IO0: now also Q5.3 (C), R15.2
- net at U1.40 (RXD0): now also U6.2 (TXD)
- net ESP32_EN: now reaches U1.45 (EN)
- net ESP32_EN: now also Q3.3 (C), R2.2
- net IRQ_ACC: now reaches U1.7 (IO3)
- net IRQ_ACC: now also U5.12 (INT1)
- net INT_MAX: now reaches U1.9 (IO5)
- net INT_MAX: now also J3.4 (Pin_4)
- new net: R3.1, U4.2 (PROG)
- new net: P1.A6 (D+), U6.5 (UD+)
- new net: P1.A7 (D-), U6.6 (UD-)
- new net: Q3.1 (B), R13.2
- new net: C6.1, J3.3 (Pin_3)
- new net: U2.11 (RESERVED), U2.7 (RESERVED), U2.8 (RESERVED)
- new net: C12.1, U3.4 (BYPASS)
- new net: C1.1, J3.2 (Pin_2)
- new net: Q5.1 (B), R14.2
- new net CHRG: Q1.1 (G), R5.2, U4.7 (~{CHRG})
- new net DTR: Q5.2 (E), R13.1, U6.13 (~{DTR})
- new net POWER_5V: C13.1, P1.A4 (VBUS), P1.A9 (VBUS), P1.B4 (VBUS), P1.B9 (VBUS), R4.1, R5.1, U4.4 (VCC), U4.8 (CE)
- new net RTS: Q3.2 (E), R14.1, U6.14 (~{RTS})
- new net STDBY: Q2.1 (G), R4.2, U4.6 (~{STDBY})
- new net VTP4: C14.1, C2.1, J2.1 (Pin_1), U3.1 (VIN), U3.3 (ON/~{OFF}), U4.5 (BAT)
- no-connect marks 0 -> 30
Other:
- moved on the sheet: U1

Commit message: edit design
Connections:
- net DTR: now also Q3.2 (E), R14.1; no longer Q5.2 (E), R13.1
- net RTS: now also Q5.2 (E), R13.1; no longer Q3.2 (E), R14.1
Changed lines of the file:
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@@
 		)
 	)
-	(label "DTR"
+	(label "RTS"
 		(at 321.31 195.58 0)
 		(fields_autoplaced yes)
@@
 		)
 	)
-	(label "RTS"
+	(label "DTR"
 		(at 321.31 214.63 0)
 		(fields_autoplaced yes)

Commit message: cajbvjadbvj
Parts:
- added J7: Conn_01x04_Pin, symbol Connector:Conn_01x04_Pin
Connections:
- net +3.3V: now also J7.2 (Pin_2)
- net GND: now also J7.1 (Pin_1)
- net I2C_SCL: now also J7.4 (Pin_4)
- net I2C_SDA: now also J7.3 (Pin_3)
Other:
- note added: "Oled"
