File: Design/wearable_device/wearable_device.kicad_pcb (KiCad board)
At the start: 2 copper layers, 2 parts, among them U1 ESP32-S3-MINI-1

Commit message: complete design pcb board
Parts:
- removed IC**: TESEOLIV3R, SamacSys_Parts:TESEOLIV3R
- added C1: 10uF, Capacitor_SMD:C_0603_1608Metric, F.Cu at (192.0, 93.8)
- added C12: 10nF, Capacitor_SMD:C_0603_1608Metric, F.Cu at (225.7, 79.5)
- added C13: 10uF, Capacitor_SMD:C_0603_1608Metric, F.Cu at (221.4, 88.5)
- added C14: 10uF, Capacitor_SMD:C_0603_1608Metric, F.Cu at (222.2, 79.5)
- added C15: 100nF, Capacitor_SMD:C_0603_1608Metric, B.Cu at (212.2, 61.5)
- added C16: 100nF, Capacitor_SMD:C_0603_1608Metric, B.Cu at (212.2, 60.0)
- added C17: 10uF, Capacitor_SMD:C_0603_1608Metric, B.Cu at (209.0, 75.5)
- added C2: 10uF, Capacitor_SMD:C_0603_1608Metric, F.Cu at (218.2, 78.5)
- added C3: 10uF, Capacitor_SMD:C_0603_1608Metric, F.Cu at (225.7, 75.7)
- added C4: 0.1uF, Capacitor_SMD:C_0603_1608Metric, F.Cu at (223.1, 67.5)
- added C5: 0.1uF, Capacitor_SMD:C_0603_1608Metric, F.Cu at (225.7, 67.5)
- added C6: 10uF, Capacitor_SMD:C_0603_1608Metric, F.Cu at (189.5, 93.8)
- added C7: 0.1uF, Capacitor_SMD:C_0603_1608Metric, F.Cu at (188.2, 73.5)
- added C8: 10uF, Capacitor_SMD:C_0603_1608Metric, F.Cu at (192.0, 73.5)
- added C9: 0.1uF, Capacitor_SMD:C_0603_1608Metric, F.Cu at (191.8, 67.7)
- added J1: Micro_SD_Card, Connector_Card:microSD_HC_Hirose_DM3D-SF, B.Cu at (220.6, 76.3)
- added J2: POWER, Connector_PinHeader_2.00mm:PinHeader_1x01_P2.00mm_Vertical, F.Cu at (225.2, 92.0)
- added J3: Conn_01x04_Pin, Connector_PinHeader_2.00mm:PinHeader_1x04_P2.00mm_Vertical, F.Cu at (193.0, 88.5)
- added J4: Conn_01x04_Pin, Connector_PinHeader_2.00mm:PinHeader_1x04_P2.00mm_Vertical, F.Cu at (188.9, 88.5)
- added J5: Conn_01x07_Pin, Connector_PinHeader_2.54mm:PinHeader_1x07_P2.54mm_Vertical, F.Cu at (194.9, 94.2)
- added J6: GND, Connector_PinHeader_2.00mm:PinHeader_1x01_P2.00mm_Vertical, F.Cu at (225.2, 95.5)
- added P1: USB_C_Plug_USB2.0, Connector_USB:USB_C_Receptacle_GCT_USB4105-xx-A_16P_TopMnt_Horizontal, F.Cu at (217.7, 95.5)
- added Q1: BSS138, Package_TO_SOT_SMD:SOT-23, F.Cu at (214.1, 80.5)
- added Q2: BSS138, Package_TO_SOT_SMD:SOT-23, F.Cu at (209.7, 80.5)
- added Q3: BC817, Package_TO_SOT_SMD:SOT-23, F.Cu at (223.7, 61.0)
- added Q5: BC817, Package_TO_SOT_SMD:SOT-23, F.Cu at (200.6, 62.4)
- added R1: 10k, Resistor_SMD:R_0603_1608Metric, B.Cu at (209.0, 84.0)
- added R10: 10k, Resistor_SMD:R_0603_1608Metric, B.Cu at (207.5, 84.0)
- added R11: 10k, Resistor_SMD:R_0603_1608Metric, B.Cu at (211.5, 84.0)
- added R12: 10k, Resistor_SMD:R_0603_1608Metric, B.Cu at (205.5, 84.0)
- added R13: 10k, Resistor_SMD:R_0603_1608Metric, F.Cu at (224.2, 64.5)
- added R14: 10k, Resistor_SMD:R_0603_1608Metric, F.Cu at (197.7, 66.5)
- added R15: 10k, Resistor_SMD:R_0603_1608Metric, F.Cu at (202.7, 66.5)
- added R16: 10k, Resistor_SMD:R_0603_1608Metric, B.Cu at (217.5, 59.5)
- added R2: 10k, Resistor_SMD:R_0603_1608Metric, F.Cu at (220.7, 59.5)
- added R3: 1.2k, Resistor_SMD:R_0603_1608Metric, F.Cu at (225.2, 89.0)
- added R4: 10k, Resistor_SMD:R_0603_1608Metric, F.Cu at (211.1, 86.5)
- added R5: 10k, Resistor_SMD:R_0603_1608Metric, F.Cu at (213.7, 86.5)
- added R6: 10k, Resistor_SMD:R_0603_1608Metric, F.Cu at (208.0, 75.0)
- added R7: 10k, Resistor_SMD:R_0603_1608Metric, F.Cu at (213.2, 75.0)
- added R8: 4.7k, Resistor_SMD:R_0603_1608Metric, B.Cu at (207.0, 69.5)
- added R9: 4.7k, Resistor_SMD:R_0603_1608Metric, B.Cu at (211.7, 69.0)
- added SW1: SW_Push, Button_Switch_SMD:SW_Tactile_SPST_NO_Straight_CK_PTS636Sx25SMTRLFS, B.Cu at (224.5, 63.0)
- added U2: L80-R, L80-R:XCVR_L80-R, B.Cu at (189.8, 69.3)
- added U3: LP2985-33DBVR, LP2985-33DBVR:SOT95P280X145-5N, F.Cu at (222.7, 77.0)
- added U4: TP4056, TP4056:SOP127P600X175-9N, F.Cu at (220.2, 83.5)
- added U5: LIS2DH12TR, LIS2DH12TR:PQFN50P200X200100-12N, B.Cu at (216.3, 63.8)
- added U6: CH340C, Package_SO:SOIC-16_3.9x9.9mm_P1.27mm, F.Cu at (203.2, 82.5)
- moved U1 51.7 mm to (211.7, 63.0)
Connections:
- net Net-(U1-GND-Pad1) renamed GND
- U1 pad 10: unconnected-(U1-IO6-Pad10) -> /MOSI_SPI2
- U1 pad 11: unconnected-(U1-IO7-Pad11) -> /CS_SPI2
- U1 pad 12: unconnected-(U1-IO8-Pad12) -> /RES_TFT
- U1 pad 13: unconnected-(U1-IO9-Pad13) -> /DC_TFT
- U1 pad 14: unconnected-(U1-IO10-Pad14) -> /BLK_TFT
- U1 pad 16: unconnected-(U1-IO12-Pad16) -> /MOSI_TFT
- U1 pad 17: unconnected-(U1-IO13-Pad17) -> /I2C_SCL
- U1 pad 18: unconnected-(U1-IO14-Pad18) -> /I2C_SDA
- U1 pad 19: unconnected-(U1-IO15-Pad19) -> /SCLK_TFT
- U1 pad 20: unconnected-(U1-IO16-Pad20) -> /CLK_SPI2
- U1 pad 21: unconnected-(U1-IO17-Pad21) -> /RXD1
- U1 pad 22: unconnected-(U1-IO18-Pad22) -> /TXD1
- U1 pad 23: unconnected-(U1-IO19-Pad23) -> /MISO_SPI2
- U1 pad 3: unconnected-(U1-3V3-Pad3) -> +3.3V
- U1 pad 33: unconnected-(U1-IO37-Pad33) -> /SG_STDBY
- U1 pad 34: unconnected-(U1-IO38-Pad34) -> /SG_CHRG
- U1 pad 35: unconnected-(U1-IO39-Pad35) -> /BTN_CONTROL
- U1 pad 39: unconnected-(U1-TXD0-Pad39) -> Net-(U1-TXD0)
- U1 pad 4: unconnected-(U1-IO0-Pad4) -> /ESP32_IO0
- U1 pad 40: unconnected-(U1-RXD0-Pad40) -> Net-(U1-RXD0)
- U1 pad 45: unconnected-(U1-EN-Pad45) -> /ESP32_EN
- U1 pad 7: unconnected-(U1-IO3-Pad7) -> /IRQ_ACC
- U1 pad 9: unconnected-(U1-IO5-Pad9) -> /INT_MAX
Routing:
- net +3.3V: track 0.00 -> 245.3 mm, vias 0 -> 16
- net /RTS: track 0.00 -> 60.5 mm, vias 0 -> 3
- net /I2C_SCL: track 0.00 -> 54.8 mm, vias 0 -> 2
- net /I2C_SDA: track 0.00 -> 52.7 mm, vias 0 -> 3
- net /DTR: track 0.00 -> 51.4 mm, vias 0 -> 3
- net /DC_TFT: track 0.00 -> 45.1 mm, vias 0 -> 2
- net /POWER_5V: track 0.00 -> 43.7 mm, vias 0 -> 2
- net /RES_TFT: track 0.00 -> 42.7 mm, vias 0 -> 1
- net /MOSI_TFT: track 0.00 -> 38.2 mm, vias 0 -> 2
- net Net-(U1-TXD0): track 0.00 -> 34.3 mm
- net Net-(U1-RXD0): track 0.00 -> 33.3 mm, vias 0 -> 2
- net /CS_SPI2: track 0.00 -> 32.7 mm, vias 0 -> 1
- net /BLK_TFT: track 0.00 -> 32.0 mm, vias 0 -> 2
- net /MOSI_SPI2: track 0.00 -> 31.0 mm, vias 0 -> 2
- net Net-(P1-D+): track 0.00 -> 30.8 mm
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- added copper zone on B.Cu, net GND
- added copper zone on F.Cu, net GND
- added copper zone on In1.Cu, net GND
- added copper zone on In2.Cu, net GND
Other:
- board outline added: 50 x 41.2 mm
- copper layers 2 -> 4
